File: PLC/plc.kicad_pcb (KiCad board)
At the start: 2 copper layers, 16 parts, among them SW1 SW_PUSH, U1 OPTO-TRANSISTOR, U3 LM7805

Commit message: plc
Parts:
- removed 0.1uF1, 0.33uF1: C, Capacitor_THT:C_Disc_D8.0mm_W2.5mm_P5.00mm
- removed 10k1: R, Resistor_THT:R_Axial_DIN0204_L3.6mm_D1.6mm_P5.08mm_Horizontal
- removed 1N4007: DIODE, Diode_THT:D_A-405_P7.62mm_Horizontal
- removed 1k1: R, Resistor_THT:R_Axial_DIN0309_L9.0mm_D3.2mm_P12.70mm_Horizontal
- removed 2N3904: NPN, Package_TO_SOT_THT:TO-92_HandSolder
- removed Vin1: CONN_2, TerminalBlock_Phoenix:TerminalBlock_Phoenix_MKDS-1,5-2-5.08_1x02_P5.08mm_Horizontal
- added A1: Arduino_Nano_v3.x, Module:Arduino_Nano, F.Cu at (91.7, 128.9)
- added C10: 1uF, Capacitor_THT:CP_Radial_D5.0mm_P2.50mm, F.Cu at (152.1, 122.7)
- added C11: 1uF, Capacitor_THT:CP_Radial_D5.0mm_P2.50mm, F.Cu at (151.3, 144.1)
- added C12: 1uF, Capacitor_THT:CP_Radial_D5.0mm_P2.50mm, F.Cu at (152.1, 163.1)
- added C2: 1uF, Capacitor_THT:CP_Radial_D5.0mm_P2.50mm, F.Cu at (152.8, 33.1)
- added C3: 1uF, Capacitor_THT:CP_Radial_D5.0mm_P2.50mm, F.Cu at (152.5, 69.0)
- added C4: 1uF, Capacitor_THT:CP_Radial_D5.0mm_P2.50mm, F.Cu at (151.6, 86.9)
- added C5: 1uF, Capacitor_THT:CP_Radial_D5.0mm_P2.50mm, F.Cu at (151.8, 105.9)
- added C6: 0.33uF1, Capacitor_THT:C_Disc_D8.0mm_W5.0mm_P5.00mm, F.Cu at (90.3, 35.2)
- added C7: 0.33uF1, Capacitor_THT:C_Disc_D8.0mm_W5.0mm_P5.00mm, F.Cu at (104.5, 35.2)
- added C8: 0.1uF1, Capacitor_THT:C_Disc_D5.0mm_W2.5mm_P2.50mm, F.Cu at (97.4, 35.4)
- added C9: 0.1uF1, Capacitor_THT:C_Disc_D5.0mm_W2.5mm_P2.50mm, F.Cu at (111.6, 35.4)
- added D10: LED, LED_THT:LED_D3.0mm, F.Cu at (134.3, 127.8)
- added D11: LED, LED_THT:LED_D3.0mm, F.Cu at (134.2, 148.0)
- added D12: LED, LED_THT:LED_D3.0mm, F.Cu at (134.5, 166.7)
- added D13: LED, LED_THT:LED_D3.0mm, F.Cu at (80.5, 57.6)
- added D14: 1N4007, Diode_THT:D_A-405_P7.62mm_Horizontal, F.Cu at (67.3, 49.4)
- added D15: LED, LED_THT:LED_D3.0mm, F.Cu at (80.0, 72.3)
- added D16: 1N4007, Diode_THT:D_A-405_P7.62mm_Horizontal, F.Cu at (66.9, 64.4)
- added D17: LED, LED_THT:LED_D3.0mm, F.Cu at (80.1, 87.3)
- added D18: 1N4007, Diode_THT:D_A-405_P7.62mm_Horizontal, F.Cu at (67.1, 79.4)
- added D19: LED, LED_THT:LED_D3.0mm, F.Cu at (79.8, 103.6)
- added D20: 1N4007, Diode_THT:D_A-405_P7.62mm_Horizontal, F.Cu at (66.9, 95.7)
- added D21: LED, LED_THT:LED_D3.0mm, F.Cu at (79.7, 123.3)
- added D22: 1N4007, Diode_THT:D_A-405_P7.62mm_Horizontal, F.Cu at (66.5, 123.0)
- added D23: LED, LED_THT:LED_D3.0mm, F.Cu at (79.5, 166.3)
- added D24: 1N4007, Diode_THT:D_A-405_P7.62mm_Horizontal, F.Cu at (67.1, 165.8)
- added D25: LED, LED_THT:LED_D3.0mm, F.Cu at (111.7, 39.7)
- added D3: 1N4007, Diode_THT:D_A-405_P7.62mm_Horizontal, F.Cu at (66.8, 144.7)
- added D4: LED, LED_THT:LED_D3.0mm, F.Cu at (134.6, 37.7)
- added D5: 1N4007, Diode_THT:D_A-405_P7.62mm_Horizontal, F.Cu at (67.4, 34.9)
- added D6: LED, LED_THT:LED_D3.0mm, F.Cu at (134.5, 54.3)
- added D7: LED, LED_THT:LED_D3.0mm, F.Cu at (135.0, 73.3)
- added D8: LED, LED_THT:LED_D3.0mm, F.Cu at (134.4, 91.2)
- added D9: LED, LED_THT:LED_D3.0mm, F.Cu at (134.1, 110.2)
- added J1: Conn_in24_0, TerminalBlock:TerminalBlock_bornier-5_P5.08mm, F.Cu at (163.6, 59.1)
- added J2: Conn_in24_1, TerminalBlock:TerminalBlock_bornier-5_P5.08mm, F.Cu at (163.6, 123.0)
- added J3: Conn_rele_0, TerminalBlock:TerminalBlock_bornier-5_P5.08mm, F.Cu at (34.7, 59.3)
- added J4: Conn_rele_1, TerminalBlock:TerminalBlock_bornier-5_P5.08mm, F.Cu at (34.7, 124.8)
- added K1: FINDER-36.11, Relay_THT:Relay_SPDT_Finder_36.11, F.Cu at (61.9, 141.1)
- added K2: FINDER-36.11, Relay_THT:Relay_SPDT_Finder_36.11, F.Cu at (62.2, 162.3)
- added K3: FINDER-36.11, Relay_THT:Relay_SPDT_Finder_36.11, F.Cu at (61.9, 119.3)
- added Q1: BC557, Package_TO_SOT_THT:TO-92_Inline, F.Cu at (72.8, 137.6)
- added Q2: BC557, Package_TO_SOT_THT:TO-92_Inline, F.Cu at (74.7, 34.9)
- added Q3: BC557, Package_TO_SOT_THT:TO-92_Inline, F.Cu at (74.1, 49.4)
- added Q4: BC557, Package_TO_SOT_THT:TO-92_Inline, F.Cu at (73.6, 64.4)
- added Q5: BC557, Package_TO_SOT_THT:TO-92_Inline, F.Cu at (73.5, 79.4)
- added Q6: BC557, Package_TO_SOT_THT:TO-92_Inline, F.Cu at (73.7, 95.7)
- added Q7: BC557, Package_TO_SOT_THT:TO-92_Inline, F.Cu at (73.6, 115.2)
- added Q8: BC557, Package_TO_SOT_THT:TO-92_Inline, F.Cu at (73.1, 158.2)
- added R10: 1k, Resistor_THT:R_Axial_DIN0204_L3.6mm_D1.6mm_P5.08mm_Horizontal, F.Cu at (141.6, 66.7)
- added R11: 1k, Resistor_THT:R_Axial_DIN0204_L3.6mm_D1.6mm_P5.08mm_Horizontal, F.Cu at (150.5, 91.3)
- added R12: 1k, Resistor_THT:R_Axial_DIN0204_L3.6mm_D1.6mm_P5.08mm_Horizontal, F.Cu at (140.8, 84.7)
- added R13: 1k, Resistor_THT:R_Axial_DIN0204_L3.6mm_D1.6mm_P5.08mm_Horizontal, F.Cu at (150.5, 110.1)
- added R14: 1k, Resistor_THT:R_Axial_DIN0204_L3.6mm_D1.6mm_P5.08mm_Horizontal, F.Cu at (140.7, 104.0)
- added R15: 1k, Resistor_THT:R_Axial_DIN0204_L3.6mm_D1.6mm_P5.08mm_Horizontal, F.Cu at (151.0, 127.5)
- added R16: 1k, Resistor_THT:R_Axial_DIN0204_L3.6mm_D1.6mm_P5.08mm_Horizontal, F.Cu at (141.0, 120.7)
- added R17: 1k, Resistor_THT:R_Axial_DIN0204_L3.6mm_D1.6mm_P5.08mm_Horizontal, F.Cu at (150.7, 148.3)
- added R18: 1k, Resistor_THT:R_Axial_DIN0204_L3.6mm_D1.6mm_P5.08mm_Horizontal, F.Cu at (141.2, 141.5)
- added R19: 1k, Resistor_THT:R_Axial_DIN0204_L3.6mm_D1.6mm_P5.08mm_Horizontal, F.Cu at (150.7, 167.3)
- added R20: 1k, Resistor_THT:R_Axial_DIN0204_L3.6mm_D1.6mm_P5.08mm_Horizontal, F.Cu at (141.4, 161.2)
- added R21: 1K, Resistor_THT:R_Axial_DIN0204_L3.6mm_D1.6mm_P5.08mm_Horizontal, F.Cu at (76.7, 54.8)
- added R22: 10k, Resistor_THT:R_Axial_DIN0204_L3.6mm_D1.6mm_P5.08mm_Horizontal, F.Cu at (71.6, 57.6)
- added R23: 1K, Resistor_THT:R_Axial_DIN0204_L3.6mm_D1.6mm_P5.08mm_Horizontal, F.Cu at (76.2, 69.8)
- added R24: 10k, Resistor_THT:R_Axial_DIN0204_L3.6mm_D1.6mm_P5.08mm_Horizontal, F.Cu at (71.1, 72.3)
- added R25: 1K, Resistor_THT:R_Axial_DIN0204_L3.6mm_D1.6mm_P5.08mm_Horizontal, F.Cu at (76.0, 84.8)
- added R26: 10k, Resistor_THT:R_Axial_DIN0204_L3.6mm_D1.6mm_P5.08mm_Horizontal, F.Cu at (70.9, 87.3)
- added R27: 1K, Resistor_THT:R_Axial_DIN0204_L3.6mm_D1.6mm_P5.08mm_Horizontal, F.Cu at (76.0, 101.0)
- added R28: 10k, Resistor_THT:R_Axial_DIN0204_L3.6mm_D1.6mm_P5.08mm_Horizontal, F.Cu at (70.9, 103.6)
- added R29: 1K, Resistor_THT:R_Axial_DIN0204_L3.6mm_D1.6mm_P5.08mm_Horizontal, F.Cu at (75.9, 120.5)
- added R3: 1K, Resistor_THT:R_Axial_DIN0204_L3.6mm_D1.6mm_P5.08mm_Horizontal, F.Cu at (75.4, 142.9)
- added R30: 10k, Resistor_THT:R_Axial_DIN0204_L3.6mm_D1.6mm_P5.08mm_Horizontal, F.Cu at (70.8, 123.3)
- added R31: 1K, Resistor_THT:R_Axial_DIN0204_L3.6mm_D1.6mm_P5.08mm_Horizontal, F.Cu at (75.7, 163.8)
- added R32: 10k, Resistor_THT:R_Axial_DIN0204_L3.6mm_D1.6mm_P5.08mm_Horizontal, F.Cu at (70.7, 166.3)
- added R33: 1k, Resistor_THT:R_Axial_DIN0204_L3.6mm_D1.6mm_P5.08mm_Horizontal, F.Cu at (115.0, 35.4)
- added R4: 10k, Resistor_THT:R_Axial_DIN0204_L3.6mm_D1.6mm_P5.08mm_Horizontal, F.Cu at (70.3, 145.5)
- added R5: 1k, Resistor_THT:R_Axial_DIN0204_L3.6mm_D1.6mm_P5.08mm_Horizontal, F.Cu at (151.6, 37.6)
- added R6: 1k, Resistor_THT:R_Axial_DIN0204_L3.6mm_D1.6mm_P5.08mm_Horizontal, F.Cu at (142.1, 30.6)
- added R7: 1k, Resistor_THT:R_Axial_DIN0204_L3.6mm_D1.6mm_P5.08mm_Horizontal, F.Cu at (151.9, 54.3)
- added R8: 1k, Resistor_THT:R_Axial_DIN0204_L3.6mm_D1.6mm_P5.08mm_Horizontal, F.Cu at (141.5, 47.8)
- added R9: 1k, Resistor_THT:R_Axial_DIN0204_L3.6mm_D1.6mm_P5.08mm_Horizontal, F.Cu at (151.6, 73.6)
- added SW2: SW_PUSH, Button_Switch_THT:SW_PUSH_6mm_H5mm, F.Cu at (129.2, 38.1)
- added SW3: SW_PUSH, Button_Switch_THT:SW_PUSH_6mm_H5mm, F.Cu at (129.3, 73.6)
- added SW4: SW_PUSH, Button_Switch_THT:SW_PUSH_6mm_H5mm, F.Cu at (129.2, 91.2)
- added SW5: SW_PUSH, Button_Switch_THT:SW_PUSH_6mm_H5mm, F.Cu at (128.9, 110.8)
- added SW6: SW_PUSH, Button_Switch_THT:SW_PUSH_6mm_H5mm, F.Cu at (129.1, 129.1)
- added SW7: SW_PUSH, Button_Switch_THT:SW_PUSH_6mm_H5mm, F.Cu at (129.2, 148.2)
- added SW8: SW_PUSH, Button_Switch_THT:SW_PUSH_6mm_H5mm, F.Cu at (129.3, 167.6)
- added U10: PC817, Package_DIP:DIP-4_W7.62mm, F.Cu at (147.5, 148.3)
- added U11: PC817, Package_DIP:DIP-4_W7.62mm, F.Cu at (147.6, 167.3)
- added U12: ~, Relay_THT:RSEIV-JMU, F.Cu at (54.1, 53.3)
- added U13: ~, Relay_THT:RSEIV-JMU, F.Cu at (53.8, 68.3)
- added U14: ~, Relay_THT:RSEIV-JMU, F.Cu at (53.8, 83.3)
- added U15: ~, Relay_THT:RSEIV-JMU, F.Cu at (53.7, 99.5)
- added U4: PC817, Package_DIP:DIP-4_W7.62mm, F.Cu at (147.9, 73.5)
- added U5: LM7812_TO220, Package_TO_SOT_THT:TO-220-3_Vertical, F.Cu at (90.3, 30.3)
- added U6: LM7805_TO220, Package_TO_SOT_THT:TO-220-3_Vertical, F.Cu at (104.5, 30.3)
- added U7: PC817, Package_DIP:DIP-4_W7.62mm, F.Cu at (147.3, 91.3)
- added U8: PC817, Package_DIP:DIP-4_W7.62mm, F.Cu at (147.0, 110.2)
- added U9: PC817, Package_DIP:DIP-4_W7.62mm, F.Cu at (147.3, 127.4)
- added con2: Vin, TerminalBlock_Phoenix:TerminalBlock_Phoenix_MKDS-1,5-2-5.08_1x02_P5.08mm_Horizontal, F.Cu at (35.5, 35.3)
- C1: footprint Capacitor_THT:C_Radial_D6.3mm_H11.0mm_P2.50mm -> Capacitor_THT:CP_Radial_D5.0mm_P2.50mm
- R1: value 1k -> 1K; footprint Resistor_THT:R_Axial_DIN0309_L9.0mm_D3.2mm_P12.70mm_Horizontal -> Resistor_THT:R_Axial_DIN0204_L3.6mm_D1.6mm_P5.08mm_Horizontal
- R2: value 1k -> 10k; footprint Resistor_THT:R_Axial_DIN0309_L9.0mm_D3.2mm_P12.70mm_Horizontal -> Resistor_THT:R_Axial_DIN0204_L3.6mm_D1.6mm_P5.08mm_Horizontal
- SW1: footprint Button_Switch_THT:SW_PUSH_6mm -> Button_Switch_THT:SW_PUSH_6mm_H5mm
- U1: value OPTO-TRANSISTOR -> PC817; footprint Package_DIP:DIP-6_W7.62mm_LongPads -> Package_DIP:DIP-4_W7.62mm
- U2: value ~ -> PC817; footprint Relay_THT:RSEIV-JMU -> Package_DIP:DIP-4_W7.62mm
- U3: value LM7805 -> ~; footprint Package_TO_SOT_THT:TO-220-3_Vertical -> Relay_THT:RSEIV-JMU
- moved U3 135.6 mm to (54.1, 38.7), turned to 180 degrees
- moved R2 100.5 mm to (71.5, 42.8)
- moved R1 97.4 mm to (76.7, 40.2), turned to 180 degrees
- moved D1 79.7 mm to (80.2, 42.8), turned to 90 degrees
- moved D2 78.9 mm to (79.0, 145.5)
- moved C1 54.1 mm to (153.0, 49.7)
- moved SW1 46.0 mm to (129.1, 54.2), turned to 180 degrees
- moved U1 43.4 mm to (148.2, 37.4), turned to 180 degrees
- moved U2 27.6 mm to (148.0, 54.0), turned to 180 degrees
Connections:
- C1 pad 1: /in_0 -> in_1
- D1 pad 1: /in_0 -> out_0
- D2 pad 1: /out_0 -> out_6
- R1 pad 1: Net-(U1-A) -> Net-(D1-K)
- R1 pad 2: /in24_0 -> GND
- R2 pad 1: Net-(D1-K) -> Net-(Q2-B)
- R2 pad 2: GND -> out_0
- SW1 pad 2: /in_0 -> in_1
- U1 pad 1: Net-(U1-A) -> Net-(R5-Pad1)
- U1 pad 3: unconnected-(U1-NC-Pad3) -> in_0
- U1 pad 4: /in_0 -> +5V
- U2 pad 1: +5V -> Net-(R7-Pad1)
- U2 pad 2: Net-(1N4007-A) -> GND
- U2 pad 3: /outR_0 -> in_1
- U2 pad 4: /pwr_R_0 -> +5V
- U3 pad 1: (no net) -> +12V
- U3 pad 2: (no net) -> Net-(D5-A)
- U3 pad 3: (no net) -> outR_0
Routing:
- net GND: track 0.00 -> 700.5 mm, vias 0 -> 1
- net +5V: track 0.00 -> 358.2 mm
- net +12V: track 0.00 -> 256.1 mm
- net in_0: track 0.00 -> 183.3 mm
- net in_1: track 0.00 -> 176.5 mm
- net in_2: track 0.00 -> 155.1 mm
- net pwr_R_1: track 0.00 -> 132.2 mm
- net in_3: track 0.00 -> 126.7 mm
- net out_0: track 0.00 -> 106.3 mm
- net in_4: track 0.00 -> 105.7 mm
- net out_1: track 0.00 -> 94.7 mm
- net in_6: track 0.00 -> 90.4 mm, vias 0 -> 1
- net in_5: track 0.00 -> 89.2 mm
- net pwr_R_0: track 0.00 -> 83.6 mm
- net Vin: track 0.00 -> 83.1 mm
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- added copper zone on B.Cu, net GND
Other:
- board text added: "PLC UTN-FRC 2023 Agustin Romero Joaquin Pappano Juan Monteros"
