File: PLC/plc.kicad_sch (KiCad schematic)
At the start: 16 parts, among them SW1 SW_PUSH, U1 OPTO-TRANSISTOR, U3 LM7805

Commit message: plc
Parts:
- removed 0.1uF1, 0.33uF1: C, Capacitor_THT:C_Disc_D8.0mm_W2.5mm_P5.00mm, symbol plc-rescue:C
- removed 10k1: R, Resistor_THT:R_Axial_DIN0204_L3.6mm_D1.6mm_P5.08mm_Horizontal, symbol plc-rescue:R
- removed 1N4007: DIODE, Diode_THT:D_A-405_P7.62mm_Horizontal, symbol plc-rescue:DIODE
- removed 1k1: R, Resistor_THT:R_Axial_DIN0309_L9.0mm_D3.2mm_P12.70mm_Horizontal, symbol plc-rescue:R
- removed 2N3904: NPN, Package_TO_SOT_THT:TO-92_HandSolder, symbol plc-rescue:NPN
- removed C1: 1uF, Capacitor_THT:C_Radial_D6.3mm_H11.0mm_P2.50mm, symbol plc-rescue:CP1
- removed D1, D2: LED, LED_THT:LED_D3.0mm, symbol plc-rescue:LED
- removed R1, R2: 1k, Resistor_THT:R_Axial_DIN0309_L9.0mm_D3.2mm_P12.70mm_Horizontal, symbol plc-rescue:R
- removed SW1: SW_PUSH, Button_Switch_THT:SW_PUSH_6mm, symbol plc-rescue:SW_PUSH
- removed U1: OPTO-TRANSISTOR, Package_DIP:DIP-6_W7.62mm_LongPads, symbol plc-rescue:OPTO-TRANSISTOR
- removed U2: ~, Relay_THT:RSEIV-JMU, symbol Relay:RSEIV-JMU
- removed U3: LM7805, Package_TO_SOT_THT:TO-220-3_Vertical, symbol plc-rescue:LM7805
- removed Vin1: CONN_2, TerminalBlock_Phoenix:TerminalBlock_Phoenix_MKDS-1,5-2-5.08_1x02_P5.08mm_Horizontal, symbol plc-rescue:CONN_2
- added A1: Arduino_Nano_v3.x, Module:Arduino_Nano, symbol MCU_Module:Arduino_Nano_v3.x
- added H1, H2, H3, H4: MountingHole, symbol Mechanical:MountingHole
- added J1: Conn_in24_0, TerminalBlock:TerminalBlock_bornier-5_P5.08mm, symbol Connector:Conn_01x05_Pin
- added J2: Conn_in24_1, TerminalBlock:TerminalBlock_bornier-5_P5.08mm, symbol Connector:Conn_01x05_Pin
- added J3: Conn_rele_0, TerminalBlock:TerminalBlock_bornier-5_P5.08mm, symbol Connector:Conn_01x05_Pin
- added J4: Conn_rele_1, TerminalBlock:TerminalBlock_bornier-5_P5.08mm, symbol Connector:Conn_01x05_Pin
Connections:
- net +5V: now also A1.30 (VIN)
- net GND: now also A1.29 (GND), A1.4 (GND), J1.1 (Pin_1), J2.1 (Pin_1)
- net in24_0: now also J1.2 (Pin_2)
- net in_0: now also A1.13 (D10)
- net outR_0: now also J3.2 (Pin_2)
- net out_0: now also A1.5 (D2)
- net pwr_R_0: now also J3.1 (Pin_1)
- new net in24_1: J1.3 (Pin_3)
- new net in24_2: J1.4 (Pin_4)
- new net in24_3: J1.5 (Pin_5)
- new net in24_4: J2.2 (Pin_2)
- new net in24_5: J2.3 (Pin_3)
- new net in24_6: J2.4 (Pin_4)
- new net in24_7: J2.5 (Pin_5)
- new net in_1: A1.14 (D11)
- new net in_2: A1.15 (D12)
- new net in_3: A1.16 (D13)
- new net in_4: A1.19 (A0)
- new net in_5: A1.20 (A1)
- new net in_6: A1.21 (A2)
- new net in_7: A1.22 (A3)
- new net outR_1: J3.3 (Pin_3)
- new net outR_2: J3.4 (Pin_4)
- new net outR_3: J3.5 (Pin_5)
- new net outR_4: J4.2 (Pin_2)
- new net outR_5: J4.3 (Pin_3)
- new net outR_6: J4.4 (Pin_4)
- new net outR_7: J4.5 (Pin_5)
- new net out_1: A1.6 (D3)
- new net out_2: A1.7 (D4)
- new net out_3: A1.8 (D5)
- new net out_4: A1.9 (D6)
- new net out_5: A1.10 (D7)
- new net out_6: A1.11 (D8)
- new net out_7: A1.12 (D9)
- new net pwr_R_1: J4.1 (Pin_1)
- no-connect marks 1 -> 0
Other:
- added sheet Inputs (inputs.kicad_sch)
- added sheet Outputs (outputs.kicad_sch)
- added sheet Power (Power.kicad_sch)
