File: Driver_transistor_tp1pot/Driver_transistor/Driver_MOSFET_IGBT.kicad_sch (KiCad schematic)
At the start: 12 parts, among them J1 Conn_01x01, J3 Conn_01x02, J4 Conn_01x02, Q5 IRF830, Q6 IRF830, Q7 IRG4BC30, T1 1:1

Commit message: actualizacion
Parts:
- R8: footprint Resistor_THT:R_Axial_DIN0207_L6.3mm_D2.5mm_P7.62mm_Horizontal -> Resistor_THT:R_Axial_Power_L20.0mm_W6.4mm_P22.40mm
Changed lines of the file:
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@@
       (effects (font (size 1.27 1.27)) (justify right))
     )
-    (property "Footprint" "Resistor_THT:R_Axial_DIN0207_L6.3mm_D2.5mm_P7.62mm_Horizontal" (at 203.708 54.61 90)
+    (property "Footprint" "Resistor_THT:R_Axial_Power_L20.0mm_W6.4mm_P22.40mm" (at 203.708 54.61 90)
       (effects (font (size 1.27 1.27)) hide)
     )
