File: pwm_ka3525/pwm_ka3525/pwm_ka3525.kicad_pcb (KiCad board)
At the start: 2 copper layers, 37.1 x 45.5 mm, 17 parts, among them J1 shutdown, J2 Conn_01x03, J3 Conn_01x03, J4 Conn_01x02, U1 UC3525

Commit message: actualizacion
Parts:
- added C3: 0.1uF, Capacitor_THT:C_Disc_D7.5mm_W2.5mm_P5.00mm, F.Cu at (169.2, 80.1)
- frec1: value 200k -> 150k
Routing:
- net GND: track 130.9 -> 132.6 mm
- net Vc: track 11.5 -> 12.9 mm
- net +12V: track 10.9 -> 11.7 mm
Changed lines of the file:
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@@
+    )
+  )
+  (footprint "Capacitor_THT:C_Disc_D7.5mm_W2.5mm_P5.00mm" (layer "F.Cu")
+    (at 169.164 80.09 -90)
+    (descr "C, Disc series, Radial, pin pitch=5.00mm, , diameter*width=7.5*2.5mm^2, Capacitor, http://www.vishay.com/docs/28535/vy2series.pdf")
+    (tags "C Disc series Radial pin pitch 5.00mm  diameter 7.5mm width 2.5mm Capacitor")
+    (property "Sheetfile" "pwm_ka3525.kicad_sch")
+    (property "Sheetname" "")
+    (property "ki_description" "Unpolarized capacitor")
+    (property "ki_keywords" "cap capacitor")
+    (attr through_hole)
+    (fp_text reference "C3" (at 2.5 -2.5 90) (layer "F.SilkS")
+        (effects (font (size 1 1) (thickness 0.15)))
+    )
+    (fp_text value "0.1uF" (at 2.5 2.5 90) (layer "F.Fab")
+        (effects (font (size 1 1) (thickness 0.15)))
+    )
+    (fp_text user "${REFERENCE}" (at 2.5 0 90) (layer "F.Fab")
+        (effects (font (size 1 1) (thickness 0.15)))
+    )
+    (fp_line (start -1.37 -1.37) (end -1.37 1.37)
+      (stroke (width 0.12) (type solid)) (layer "F.SilkS"))
+    (fp_line (start -1.37 -1.37) (end 6.37 -1.37)
+      (stroke (width 0.12) (type solid)) (layer "F.SilkS"))
+    (fp_line (start -1.37 1.37) (end 6.37 1.37)
+      (stroke (width 0.12) (type solid)) (layer "F.SilkS"))
+    (fp_line (start 6.37 -1.37) (end 6.37 1.37)
+      (stroke (width 0.12) (type solid)) (layer "F.SilkS"))
+    (fp_line (start -1.5 -1.5) (end -1.5 1.5)
+      (stroke (width 0.05) (type solid)) (layer "F.CrtYd"))
+    (fp_line (start -1.5 1.5) (end 6.5 1.5)
+      (stroke (width 0.05) (type solid)) (layer "F.CrtYd"))
+    (fp_line (start 6.5 -1.5) (end -1.5 -1.5)
+      (stroke (width 0.05) (type solid)) (layer "F.CrtYd"))
+    (fp_line (start 6.5 1.5) (end 6.5 -1.5)
+      (stroke (width 0.05) (type solid)) (layer "F.CrtYd"))
+    (fp_line (start -1.25 -1.25) (end -1.25 1.25)
+      (stroke (width 0.1) (type solid)) (layer "F.Fab"))
+    (fp_line (start -1.25 1.25) (end 6.25 1.25)
+      (stroke (width 0.1) (type solid)) (layer "F.Fab"))
+    (fp_line (start 6.25 -1.25) (end -1.25 -1.25)
+      (stroke (width 0.1) (type solid)) (layer "F.Fab"))
+    (fp_line (start 6.25 1.25) (end 6.25 -1.25)
+      (stroke (width 0.1) (type solid)) (layer "F.Fab"))
+    (pad "1" thru_hole circle (at 0 0 270) (size 2 2) (drill 1) (layers "*.Cu" "*.Mask")
+      (net 7 "+12V") (pintype "passive"))
+    (pad "2" thru_hole circle (at 5 0 270) (size 2 2) (drill 1) (layers "*.Cu" "*.Mask")
+      (net 2 "GND") (pintype "passive"))
+    (model "${KICAD6_3DMODEL_DIR}/Capacitor_THT.3dshapes/C_Disc_D7.5mm_W2.5mm_P5.00mm.wrl"
+      (offset (xyz 0 0 0))
+      (scale (xyz 1 1 1))
+      (rotate (xyz 0 0 0))
     )
   )
@@
         (effects (font (size 1 1) (thickness 0.15)))
     )
-    (fp_text value "200k" (at -2.54 2.34 90) (layer "F.Fab")
+    (fp_text value "150k" (at -2.54 2.34 90) (layer "F.Fab")
         (effects (font (size 1 1) (thickness 0.15)))
     )
@@
   (segment (start 142.2959 103.9419) (end 144.018 105.664) (width 1) (layer "B.Cu") (net 2))
   (segment (start 172.174001 93.421999) (end 167.260639 93.421999) (width 1) (layer "B.Cu") (net 2))
+  (segment (start 169.164 85.09) (end 170.174415 86.100415) (width 1) (layer "B.Cu") (net 2))
   (segment (start 174.701999 93.421999) (end 167.260639 93.421999) (width 1) (layer "B.Cu") (net 2))
   (segment (start 158.922719 111.252) (end 155.448 111.252) (width 1) (layer "B.Cu") (net 2))
@@
   (segment (start 155.448 111.252) (end 149.606 111.252) (width 1) (layer "B.Cu") (net 2))
   (segment (start 172.015349 107.696) (end 175.514 104.197349) (width 1) (layer "B.Cu") (net 2))
+  (segment (start 170.174415 86.100415) (end 170.174415 86.36) (width 1) (layer "B.Cu") (net 2))
   (segment (start 149.606 111.252) (end 144.018 105.664) (width 1) (layer "B.Cu") (net 2))
   (segment (start 170.174415 86.36) (end 165.724415 90.81) (width 1) (layer "B.Cu") (net 2))
@@
   (segment (start 172.87 70.394) (end 175.514 73.038) (width 1) (layer "B.Cu") (net 6))
   (segment (start 172.87 70.394) (end 166.37 70.394) (width 1) (layer "B.Cu") (net 6))
-  (segment (start 169.926 79.248) (end 172.886 79.248) (width 1) (layer "B.Cu") (net 7))
-  (segment (start 163.712 83.19) (end 165.984 83.19) (width 1) (layer "B.Cu") (net 7))
-  (segment (start 165.984 83.19) (end 169.926 79.248) (width 1) (layer "B.Cu") (net 7))
+  (segment (start 172.974 79.16) (end 170.094 79.16) (width 1) (layer "B.Cu") (net 7))
+  (segment (start 166.878 81.534) (end 166.878 80.518) (width 1) (layer "B.Cu") (net 7))
+  (segment (start 165.222 83.19) (end 166.878 81.534) (width 1) (layer "B.Cu") (net 7))
+  (segment (start 163.712 83.19) (end 165.222 83.19) (width 1) (layer "B.Cu") (net 7))
+  (segment (start 166.878 80.518) (end 167.306 80.09) (width 1) (layer "B.Cu") (net 7))
+  (segment (start 170.094 79.16) (end 169.164 80.09) (width 1) (layer "B.Cu") (net 7))
   (segment (start 172.886 79.248) (end 172.974 79.16) (width 1) (layer "B.Cu") (net 7))
+  (segment (start 167.306 80.09) (end 169.164 80.09) (width 1) (layer "B.Cu") (net 7))
+  (segment (start 164.968 88.27) (end 166.624 86.614) (width 1) (layer "B.Cu") (net 8))
+  (segment (start 166.624 84.328) (end 168.192 82.76) (width 1) (layer "B.Cu") (net 8))
   (segment (start 163.712 88.27) (end 164.968 88.27) (width 1) (layer "B.Cu") (net 8))
-  (segment (start 170.478 82.76) (end 172.974 82.76) (width 1) (layer "B.Cu") (net 8))
-  (segment (start 164.968 88.27) (end 170.478 82.76) (width 1) (layer "B.Cu") (net 8))
+  (segment (start 166.624 86.614) (end 166.624 84.328) (width 1) (layer "B.Cu") (net 8))
+  (segment (start 168.192 82.76) (end 172.974 82.76) (width 1) (layer "B.Cu") (net 8))
   (segment (start 167.93932 96.222) (end 172.974 96.222) (width 1) (layer "B.Cu") (net 9))
   (segment (start 165.06732 93.35) (end 167.93932 96.222) (width 1) (layer "B.Cu") (net 9))
