File: pic12f629/pic12f629/pic12f629.kicad_sch (KiCad schematic)
At the start: 8 parts, among them J1 Conn_02x01, J2 pickit, J3 uart, U1 PIC12F629-ISN

Commit message: OscHartley
Parts:
- added R3: R, Resistor_THT:R_Axial_DIN0207_L6.3mm_D2.5mm_P10.16mm_Horizontal, symbol Device:R
- J1: value Conn_02x01 -> Boton
Connections:
- net GND: now also R3.2
- net at BZ1.1 (-), U1.2 (GP5): now also R3.1
Other:
- moved on the sheet: J2, J3
