File: Oscilador Hartley/Oscilador_Hartley/Oscilador_Hartley.kicad_pcb (KiCad board)
At the start: 2 copper layers, 57.1 x 30 mm, 20 parts, among them J1 in, J2 Conn_01x01, J3 Conn_01x01, Q1 mpsh10

Commit message: act
Parts:
- moved J2 93.5 mm to (85.4, 42.3)
- moved C1 92.4 mm to (52.7, 46.7)
- moved C'1 92.4 mm to (45.8, 46.7)
- moved C'3 92.4 mm to (62.8, 47.0)
- moved C2 92.4 mm to (62.8, 38.4)
- moved C3 92.4 mm to (71.0, 47.0)
- moved H1 92.4 mm to (32.6, 28.9)
- moved H2 92.4 mm to (32.6, 54.3)
- moved J1 92.4 mm to (37.0, 38.2)
- moved J3 92.4 mm to (85.4, 51.0)
- moved L1 92.4 mm to (71.0, 43.1)
- moved L2 92.4 mm to (76.3, 38.3)
- moved R'2 92.4 mm to (49.6, 38.3)
- moved R1 92.4 mm to (36.9, 29.9)
- moved R2 92.4 mm to (49.6, 35.0)
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Connections:
- Q1 pad 2: Net-(Q1-E) -> Net-(Q1-C)
- Q1 pad 3: Net-(Q1-C) -> Net-(Q1-E)
