File: Oscilador Hartley/Oscilador_Hartley/Oscilador_Hartley.kicad_sch (KiCad schematic)
At the start: 20 parts, among them J1 in, J2 Conn_01x01, J3 Conn_01x01, Q1 mpsh10

Commit message: act
Connections:
- net at C4.1, L1.2, L2.1: now also Q1.3 (E); no longer Q1.2 (E)
- net at C'1.1, C1.1, R1.2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: now also Q1.2 (C); no longer Q1.3 (C)
Changed lines of the file:
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@@
     )
     (pin "1")
+    (pin "3")
     (pin "2")
-    (pin "3")
     (instances
       (project "Oscilador_Hartley"
