File: fuente_conmutada/trafo.kicad_sch (KiCad schematic)
At the start: 10 parts, among them J4 in_trafo, J4 out_R, T1 Transformer_1P_SS

Commit message: fc_v1
Parts:
- added D7: LED, LED_THT:LED_D5.0mm, symbol Device:LED
- added H1, H2, H3, H4: MountingHole, MountingHole:MountingHole_2.2mm_M2_DIN965_Pad, symbol Mechanical:MountingHole
- added R2: 22k, Resistor_THT:R_Axial_DIN0207_L6.3mm_D2.5mm_P7.62mm_Horizontal, symbol Device:R
- J4: footprint TerminalBlock_Altech:Altech_AK300_1x02_P5.00mm_45-Degree -> Connector_Phoenix_MC_HighVoltage:PhoenixContact_MC_1,5_2-G-5.08_1x02_P5.08mm_Horizontal
- L1: footprint (none) -> Inductor_THT:L_Toroid_Vertical_L16.8mm_W9.2mm_P7.10mm_Vishay_TJ3
- T1: footprint (none) -> Transformer_THT:Transformer_Breve_TEZ-22x24
Connections:
- net GNDREF: now also D7.1 (K)
- net at C1.1, J4.1 (Pin_1), L1.2: now also R2.2
- new net: D7.2 (A), R2.1
