File: fuente_conmutada/rectificador_12v.kicad_sch (KiCad schematic)
At the start: 7 parts, among them J4 Conn_01x02, J4 out_12v

Commit message: fc_v1
Parts:
- removed J4: out_12v, Connector_Phoenix_MC_HighVoltage:PhoenixContact_MC_1,5_2-G-5.08_1x02_P5.08mm_Horizontal, symbol Connector_Generic:Conn_01x02
Connections:
- net at J4.1 (Pin_1): now also D1.3; no longer D1.2
- net at J4.2 (Pin_2): now also D1.2; no longer D1.3
Other:
- moved on the sheet: J4
Changed lines of the file:
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@@
   (junction (at 158.75 91.44) (diameter 0) (color 0 0 0 0)
-  )
-  (junction (at 172.72 69.85) (diameter 0) (color 0 0 0 0)
   )
   (junction (at 166.37 91.44) (diameter 0) (color 0 0 0 0)
   )
   (junction (at 166.37 69.85) (diameter 0) (color 0 0 0 0)
-  )
-  (junction (at 172.72 91.44) (diameter 0) (color 0 0 0 0)
   )
   (wire (pts (xy 158.75 69.85) (xy 158.75 77.47))
@@
   )
   (wire (pts (xy 97.79 78.74) (xy 97.79 71.12))
-    (stroke (width 0) (type default))
-  )
-  (wire (pts (xy 172.72 91.44) (xy 184.15 91.44))
     (stroke (width 0) (type default))
   )
@@
     (stroke (width 0) (type default))
   )
+  (wire (pts (xy 93.98 81.28) (xy 97.79 81.28))
+    (stroke (width 0) (type default))
+  )
   (wire (pts (xy 148.59 88.9) (xy 148.59 91.44))
     (stroke (width 0) (type default))
   )
   (wire (pts (xy 113.03 90.17) (xy 113.03 87.63))
-    (stroke (width 0) (type default))
-  )
-  (wire (pts (xy 184.15 82.55) (xy 190.5 82.55))
     (stroke (width 0) (type default))
   )
@@
     (stroke (width 0) (type default))
   )
-  (wire (pts (xy 93.98 81.28) (xy 97.79 81.28))
-    (stroke (width 0) (type default))
-  )
   (wire (pts (xy 172.72 85.09) (xy 172.72 91.44))
-    (stroke (width 0) (type default))
-  )
-  (wire (pts (xy 93.98 78.74) (xy 97.79 78.74))
     (stroke (width 0) (type default))
   )
@@
     (stroke (width 0) (type default))
   )
-  (wire (pts (xy 184.15 69.85) (xy 172.72 69.85))
-    (stroke (width 0) (type default))
-  )
   (wire (pts (xy 158.75 91.44) (xy 166.37 91.44))
-    (stroke (width 0) (type default))
-  )
-  (wire (pts (xy 184.15 80.01) (xy 190.5 80.01))
-    (stroke (width 0) (type default))
-  )
-  (wire (pts (xy 184.15 80.01) (xy 184.15 69.85))
     (stroke (width 0) (type default))
   )
@@
     (stroke (width 0) (type default))
   )
-  (wire (pts (xy 184.15 82.55) (xy 184.15 91.44))
+  (wire (pts (xy 93.98 78.74) (xy 97.79 78.74))
     (stroke (width 0) (type default))
   )
@@
     (stroke (width 0) (type default))
   )
-  (symbol (lib_id "Connector_Generic:Conn_01x02") (at 88.9 81.28 180) (unit 1)
-    (in_bom yes) (on_board yes) (dnp no) (fields_autoplaced)
-    (property "Reference" "J4" (at 88.9 73.66 0)
+  (symbol (lib_id "Connector_Generic:Conn_01x02") (at 88.9 78.74 0) (mirror y) (unit 1)
+    (in_bom yes) (on_board yes) (dnp no)
+    (property "Reference" "J4" (at 88.9 86.36 0)
       (effects (font (size 1.27 1.27)))
     )
-    (property "Value" "Conn_01x02" (at 88.9 76.2 0)
+    (property "Value" "Conn_01x02" (at 88.9 83.82 0)
       (effects (font (size 1.27 1.27)))
     )
-    (property "Footprint" "TerminalBlock_Altech:Altech_AK300_1x02_P5.00mm_45-Degree" (at 88.9 81.28 0)
+    (property "Footprint" "TerminalBlock_Altech:Altech_AK300_1x02_P5.00mm_45-Degree" (at 88.9 78.74 0)
       (effects (font (size 1.27 1.27)) hide)
     )
-    (property "Datasheet" "~" (at 88.9 81.28 0)
+    (property "Datasheet" "~" (at 88.9 78.74 0)
       (effects (font (size 1.27 1.27)) hide)
     )
@@
         )
       )
-    )
-  )
-  (symbol (lib_id "Connector_Generic:Conn_01x02") (at 195.58 82.55 0) (mirror x) (unit 1)
-    (in_bom yes) (on_board yes) (dnp no)
-    (property "Reference" "J4" (at 198.12 81.915 0)
-      (effects (font (size 1.27 1.27)) (justify left))
-    )
-    (property "Value" "out_12v" (at 198.12 79.375 0)
-      (effects (font (size 1.27 1.27)) (justify left))
-    )
-    (property "Footprint" "Connector_Phoenix_MC_HighVoltage:PhoenixContact_MC_1,5_2-G-5.08_1x02_P5.08mm_Horizontal" (at 195.58 82.55 0)
-      (effects (font (size 1.27 1.27)) hide)
-    )
-    (property "Datasheet" "~" (at 195.58 82.55 0)
-      (effects (font (size 1.27 1.27)) hide)
-    )
-    (pin "1")
-    (pin "2")
-    (instances
-      (project "fuente_conmutada"
-        (path "/ea49c21e-f169-43d4-aeb6-478b59f13c59"
-          (reference "J4") (unit 1)
-        )
-        (path "/ea49c21e-f169-43d4-aeb6-478b59f13c59/83fe62b2-f5a2-4b35-863d-7486a6323ffd"
-          (reference "J7") (unit 1)
-        )
-      )

Commit message: fc_v1
Parts:
- C1: value 1nF -> 1000uF
- C1: value 1nF -> 100nF; footprint Capacitor_THT:CP_Radial_D8.0mm_P5.00mm -> Capacitor_THT:C_Disc_D7.5mm_W5.0mm_P5.00mm
- J4: value Conn_01x02 -> 12v _in
- R2: value 22k -> 1k
Changed lines of the file:
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@@
       (effects (font (size 1.27 1.27)))
     )
-    (property "Value" "Conn_01x02" (at 88.9 83.82 0)
+    (property "Value" "12v _in" (at 88.9 83.82 0)
       (effects (font (size 1.27 1.27)))
     )
@@
       (effects (font (size 1.27 1.27)) (justify left))
     )
-    (property "Value" "1nF" (at 162.56 83.185 0)
+    (property "Value" "1000uF" (at 162.56 83.185 0)
       (effects (font (size 1.27 1.27)) (justify left))
     )
@@
       (effects (font (size 1.27 1.27)) (justify right))
     )
-    (property "Value" "22k" (at 151.13 76.835 0)
+    (property "Value" "1k" (at 151.13 76.835 0)
       (effects (font (size 1.27 1.27)) (justify right))
     )
@@
       (effects (font (size 1.27 1.27)) (justify left))
     )
-    (property "Value" "1nF" (at 176.53 83.185 0)
-      (effects (font (size 1.27 1.27)) (justify left))
-    )
-    (property "Footprint" "Capacitor_THT:CP_Radial_D8.0mm_P5.00mm" (at 173.6852 85.09 0)
-      (effects (font (size 1.27 1.27)) hide)
-    )
+    (property "Value" "100nF" (at 176.53 83.185 0)
+      (effects (font (size 1.27 1.27)) (justify left))
+    )
+    (property "Footprint" "Capacitor_THT:C_Disc_D7.5mm_W5.0mm_P5.00mm" (at 173.6852 85.09 0)
+      (effects (font (size 1.27 1.27)) hide)
+    )
