File: fuente_conmutada/rectificador_entrada.kicad_sch (KiCad schematic)
At the start: 22 parts, among them J3 out_pwr, J4 in_red

Commit message: fc_v1
Parts:
- removed J3: out_pwr, Connector_Phoenix_MC_HighVoltage:PhoenixContact_MC_1,5_3-G-5.08_1x03_P5.08mm_Horizontal, symbol Connector_Generic:Conn_01x03
- added J16: in_pwr, Connector_Phoenix_MC_HighVoltage:PhoenixContact_MC_1,5_4-G-5.08_1x04_P5.08mm_Horizontal, symbol Connector_Generic:Conn_01x04
Connections:
- net 155V: now also J16.3 (Pin_3)
- net 310V: now also J16.4 (Pin_4)
- net GNDPWR renamed GND
- net GND: now also J16.1 (Pin_1)
- new net +12V: J16.2 (Pin_2)
Changed lines of the file:
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@@
   (junction (at 193.04 39.37) (diameter 0) (color 0 0 0 0)
   )
+  (junction (at 254 64.77) (diameter 0) (color 0 0 0 0)
+  )
   (junction (at 209.55 39.37) (diameter 0) (color 0 0 0 0)
   )
@@
     (stroke (width 0) (type default))
   )
+  (wire (pts (xy 259.08 62.23) (xy 238.76 62.23))
+    (stroke (width 0) (type default))
+  )
   (wire (pts (xy 156.21 109.22) (xy 158.75 109.22))
     (stroke (width 0) (type default))
@@
     (stroke (width 0) (type default))
   )
+  (wire (pts (xy 238.76 62.23) (xy 238.76 60.96))
+    (stroke (width 0) (type default))
+  )
   (wire (pts (xy 180.34 59.69) (xy 180.34 67.31))
     (stroke (width 0) (type default))
   )
-  (wire (pts (xy 250.19 59.69) (xy 256.54 59.69))
+  (wire (pts (xy 246.38 64.77) (xy 246.38 71.12))
+    (stroke (width 0) (type default))
+  )
+  (wire (pts (xy 250.19 59.69) (xy 259.08 59.69))
     (stroke (width 0) (type default))
   )
@@
     (stroke (width 0) (type default))
   )
+  (wire (pts (xy 254 64.77) (xy 254 71.12))
+    (stroke (width 0) (type default))
+  )
   (wire (pts (xy 130.81 109.22) (xy 130.81 114.3))
     (stroke (width 0) (type default))
@@
     (stroke (width 0) (type default))
   )
-  (wire (pts (xy 250.19 62.23) (xy 256.54 62.23))
-    (stroke (width 0) (type default))
-  )
   (wire (pts (xy 209.55 58.42) (xy 209.55 63.5))
     (stroke (width 0) (type default))
@@
     (stroke (width 0) (type default))
   )
-  (wire (pts (xy 250.19 57.15) (xy 256.54 57.15))
+  (wire (pts (xy 250.19 57.15) (xy 259.08 57.15))
     (stroke (width 0) (type default))
   )
@@
     (stroke (width 0) (type default))
   )
+  (wire (pts (xy 254 64.77) (xy 246.38 64.77))
+    (stroke (width 0) (type default))
+  )
   (wire (pts (xy 158.75 114.3) (xy 165.1 114.3))
     (stroke (width 0) (type default))
@@
     (stroke (width 0) (type default))
   )
+  (wire (pts (xy 259.08 64.77) (xy 254 64.77))
+    (stroke (width 0) (type default))
+  )
   (wire (pts (xy 219.71 81.28) (xy 219.71 83.82))
     (stroke (width 0) (type default))
@@
   )
   (wire (pts (xy 64.77 46.99) (xy 64.77 57.15))
-    (stroke (width 0) (type default))
-  )
-  (wire (pts (xy 250.19 62.23) (xy 250.19 67.31))
     (stroke (width 0) (type default))
   )
@@
     )
   )
+  (symbol (lib_id "Connector_Generic:Conn_01x04") (at 264.16 62.23 0) (mirror x) (unit 1)
+    (in_bom yes) (on_board yes) (dnp no)
+    (property "Reference" "J16" (at 266.7 61.595 0)
+      (effects (font (size 1.27 1.27)) (justify left))
+    )
+    (property "Value" "in_pwr" (at 266.7 59.055 0)
+      (effects (font (size 1.27 1.27)) (justify left))
+    )
+    (property "Footprint" "Connector_Phoenix_MC_HighVoltage:PhoenixContact_MC_1,5_4-G-5.08_1x04_P5.08mm_Horizontal" (at 264.16 62.23 0)
+      (effects (font (size 1.27 1.27)) hide)
+    )
+    (property "Datasheet" "~" (at 264.16 62.23 0)
+      (effects (font (size 1.27 1.27)) hide)
+    )
+    (pin "1")
+    (pin "2")
+    (pin "3")
+    (pin "4")
+    (instances
+      (project "fuente_conmutada"
+        (path "/ea49c21e-f169-43d4-aeb6-478b59f13c59/c8ee19b0-8cff-4830-b053-caaaff7dfdd3"
+          (reference "J16") (unit 1)
+        )
+        (path "/ea49c21e-f169-43d4-aeb6-478b59f13c59/48bdaea1-a679-4613-9073-8ffb2b3bc0e4"
+          (reference "J7") (unit 1)
+        )
+      )
+    )
+  )
   (symbol (lib_id "Mechanical:MountingHole") (at 41.91 106.68 0) (unit 1)
     (in_bom yes) (on_board yes) (dnp no) (fields_autoplaced)
@@
     )
   )
-  (symbol (lib_id "power:GNDPWR") (at 250.19 67.31 0) (unit 1)
-    (in_bom yes) (on_board yes) (dnp no) (fields_autoplaced)
-    (property "Reference" "#PWR021" (at 250.19 72.39 0)
-      (effects (font (size 1.27 1.27)) hide)
-    )
-    (property "Value" "GNDPWR" (at 250.063 72.39 0)
-      (effects (font (size 1.27 1.27)))
-    )
-    (property "Footprint" "" (at 250.19 68.58 0)
-      (effects (font (size 1.27 1.27)) hide)
-    )
-    (property "Datasheet" "" (at 250.19 68.58 0)
+  (symbol (lib_id "power:GNDPWR") (at 254 71.12 0) (unit 1)
+    (in_bom yes) (on_board yes) (dnp no) (fields_autoplaced)
+    (property "Reference" "#PWR021" (at 254 76.2 0)
+      (effects (font (size 1.27 1.27)) hide)
+    )
+    (property "Value" "GNDPWR" (at 253.873 76.2 0)
+      (effects (font (size 1.27 1.27)))
+    )
+    (property "Footprint" "" (at 254 72.39 0)
+      (effects (font (size 1.27 1.27)) hide)
+    )
+    (property "Datasheet" "" (at 254 72.39 0)
       (effects (font (size 1.27 1.27)) hide)
     )
@@
     )
   )
-  (symbol (lib_id "Connector_Generic:Conn_01x03") (at 261.62 59.69 0) (mirror x) (unit 1)
-    (in_bom yes) (on_board yes) (dnp no)
-    (property "Reference" "J3" (at 264.16 60.325 0)
-      (effects (font (size 1.27 1.27)) (justify left))
-    )
-    (property "Value" "out_pwr" (at 264.16 57.785 0)
-      (effects (font (size 1.27 1.27)) (justify left))
-    )
-    (property "Footprint" "Connector_Phoenix_MC_HighVoltage:PhoenixContact_MC_1,5_3-G-5.08_1x03_P5.08mm_Horizontal" (at 261.62 59.69 0)
-      (effects (font (size 1.27 1.27)) hide)
-    )
-    (property "Datasheet" "~" (at 261.62 59.69 0)
-      (effects (font (size 1.27 1.27)) hide)
-    )
-    (pin "1")
-    (pin "2")
-    (pin "3")
-    (instances
-      (project "fuente_conmutada"
-        (path "/ea49c21e-f169-43d4-aeb6-478b59f13c59"
-          (reference "J3") (unit 1)
-        )
-        (path "/ea49c21e-f169-43d4-aeb6-478b59f13c59/5275eb23-ead0-41a6-ad30-16f3b7375232"
-          (reference "J3") (unit 1)
-        )
-        (path "/ea49c21e-f169-43d4-aeb6-478b59f13c59/48bdaea1-a679-4613-9073-8ffb2b3bc0e4"
-          (reference "J8") (unit 1)
-        )
-      )
-    )
-  )
   (symbol (lib_id "Device:R") (at 193.04 54.61 180) (unit 1)
     (in_bom yes) (on_board yes) (dnp no) (fields_autoplaced)
@@
     )
   )
+  (symbol (lib_id "power:GND") (at 246.38 71.12 0) (unit 1)
+    (in_bom yes) (on_board yes) (dnp no) (fields_autoplaced)
+    (property "Reference" "#PWR02" (at 246.38 77.47 0)
+      (effects (font (size 1.27 1.27)) hide)
+    )
+    (property "Value" "GND" (at 246.38 76.2 0)
+      (effects (font (size 1.27 1.27)))
+    )
+    (property "Footprint" "" (at 246.38 71.12 0)
+      (effects (font (size 1.27 1.27)) hide)
+    )
+    (property "Datasheet" "" (at 246.38 71.12 0)
+      (effects (font (size 1.27 1.27)) hide)
+    )
+    (pin "1")
+    (instances
+      (project "fuente_conmutada"
+        (path "/ea49c21e-f169-43d4-aeb6-478b59f13c59"
+          (reference "#PWR02") (unit 1)
+        )
+        (path "/ea49c21e-f169-43d4-aeb6-478b59f13c59/5275eb23-ead0-41a6-ad30-16f3b7375232"
+          (reference "#PWR02") (unit 1)
+        )
+        (path "/ea49c21e-f169-43d4-aeb6-478b59f13c59/83fe62b2-f5a2-4b35-863d-7486a6323ffd"
+          (reference "#PWR014") (unit 1)
+        )
+        (path "/ea49c21e-f169-43d4-aeb6-478b59f13c59/48bdaea1-a679-4613-9073-8ffb2b3bc0e4"
+          (reference "#PWR035") (unit 1)
+        )
+      )
+    )
+  )
   (symbol (lib_id "Device:D") (at 137.16 119.38 180) (unit 1)
     (in_bom yes) (on_board yes) (dnp no) (fields_autoplaced)
@@
         )
       )
+    )
+  )
+  (symbol (lib_id "power:+12V") (at 238.76 60.96 0) (unit 1)
+    (in_bom yes) (on_board yes) (dnp no) (fields_autoplaced)
+    (property "Reference" "#PWR013" (at 238.76 64.77 0)
+      (effects (font (size 1.27 1.27)) hide)
+    )
+    (property "Value" "+12V" (at 238.76 57.15 0)
+      (effects (font (size 1.27 1.27)))
+    )
+    (property "Footprint" "" (at 238.76 60.96 0)
+      (effects (font (size 1.27 1.27)) hide)
+    )
+    (property "Datasheet" "" (at 238.76 60.96 0)
+      (effects (font (size 1.27 1.27)) hide)
+    )
+    (pin "1")
+    (instances
+      (project "fuente_conmutada"
+        (path "/ea49c21e-f169-43d4-aeb6-478b59f13c59"
+          (reference "#PWR013") (unit 1)
+        )
+        (path "/ea49c21e-f169-43d4-aeb6-478b59f13c59/83fe62b2-f5a2-4b35-863d-7486a6323ffd"
+          (reference "#PWR017") (unit 1)
+        )
+        (path "/ea49c21e-f169-43d4-aeb6-478b59f13c59/48bdaea1-a679-4613-9073-8ffb2b3bc0e4"
+          (reference "#PWR036") (unit 1)
+        )
+      )

Commit message: fc_v1
Parts:
- added J12, J9: pin, Connector_Pin:Pin_D1.3mm_L11.0mm_LooseFit, symbol Connector:Conn_01x01_Pin
- added RV1: Varistor, Varistor:RV_Disc_D12mm_W3.9mm_P7.5mm, symbol Device:Varistor
- C1: value 100n -> 10n
- C1: footprint Capacitor_THT:CP_Radial_D24.0mm_P10.00mm_SnapIn -> Capacitor_THT:CP_Radial_D35.0mm_P9mm
- J16: value in_pwr -> out_pwr
Connections:
- net Neutro: now also RV1.2
- net at C1.1, FL1.1, J4.2 (Pin_2): now also J9.1 (Pin_1)
- net at C1.2, FL1.3, J4.1 (Pin_1): now also J12.1 (Pin_1)
- net at F1.2, TH1.1: now also RV1.1
Other:
- moved on the sheet: H1, H2, H3, H4
