File: fuente_conmutada/driver.kicad_sch (KiCad schematic)
At the start: 17 parts, among them J2 pwm_power, J3 in_pwr, J3 pwm_señal, J4 in_12v, J4 trafo, Q1 IRF740, Q2 IRF740, U2 IR2110

Commit message: fc_v1
Parts:
- removed J3: in_pwr, Connector_Phoenix_MC_HighVoltage:PhoenixContact_MC_1,5_3-G-5.08_1x03_P5.08mm_Horizontal, symbol Connector_Generic:Conn_01x03
- added H1, H2, H3, H4: MountingHole, MountingHole:MountingHole_2.2mm_M2_DIN965_Pad, symbol Mechanical:MountingHole
- added J16: in_pwr, Connector_Phoenix_MC_HighVoltage:PhoenixContact_MC_1,5_4-G-5.08_1x04_P5.08mm_Horizontal, symbol Connector_Generic:Conn_01x04
- D3: footprint Diode_THT:D_A-405_P12.70mm_Horizontal -> Diode_THT:D_A-405_P10.16mm_Horizontal
- J4: value in_12v -> fan; footprint TerminalBlock_Altech:Altech_AK300_1x02_P5.00mm_45-Degree -> Connector_Wire:SolderWire-0.1sqmm_1x02_P3.6mm_D0.4mm_OD1mm
- J4: footprint TerminalBlock_Altech:Altech_AK300_1x02_P5.00mm_45-Degree -> Connector_Phoenix_MC_HighVoltage:PhoenixContact_MC_1,5_2-G-5.08_1x02_P5.08mm_Horizontal
Connections:
- net GNDPWR is gone; now on net GND: Q2.3 (S), R6.2
- net +12V: now also J16.3 (Pin_3)
- net 155V: now also J4.1 (Pin_1), J16.2 (Pin_2); no longer J4.2 (Pin_2)
- net 310V: now also J16.1 (Pin_1)
- net GND: now also J16.4 (Pin_4)
- net VS: now also J4.2 (Pin_2); no longer J4.1 (Pin_1)
Other:
- moved on the sheet: J4

Commit message: fc_v1
Parts:
- added J17: in_pwr, Connector_JST:JST_EH_B4B-EH-A_1x04_P2.50mm_Vertical, symbol Connector_Generic:Conn_01x04
- added J19: montage, Connector_PinHeader_2.54mm:PinHeader_1x10_P2.54mm_Vertical, symbol Connector:Conn_01x10_Socket
- J4: footprint Connector_Wire:SolderWire-0.1sqmm_1x02_P3.6mm_D0.4mm_OD1mm -> Connector_JST:JST_EH_B2B-EH-A_1x02_P2.50mm_Vertical
- R6: value 1k -> 10k
- R6: footprint Resistor_THT:R_Axial_DIN0207_L6.3mm_D2.5mm_P7.62mm_Horizontal -> Resistor_THT:R_Axial_DIN0207_L6.3mm_D2.5mm_P10.16mm_Horizontal
Connections:
- net +12V: now also J17.1 (Pin_1)
- net 310V: now also J19.2 (Pin_2)
- net GND: now also J17.2 (Pin_2), J19.10 (Pin_10)
- net OutA: now also J17.3 (Pin_3)
- net OutB: now also J17.4 (Pin_4)
- net VS: now also J19.3 (Pin_3), J19.4 (Pin_4), J19.9 (Pin_9)
- net 1a: now reaches D9.2 (A), Q1.1 (G), R6.1, R6.2
- net 1a: now also J19.1 (Pin_1)
- net 1b: now reaches D10.2 (A), Q2.1 (G), R6.1, R6.2
- net 1b: now also J19.7 (Pin_7), J19.8 (Pin_8)
- no-connect marks 0 -> 2

Commit message: fc_v1
Connections:
- net 1b: no longer J19.7 (Pin_7)
- no-connect marks 2 -> 3
Changed lines of the file:
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@@
   (junction (at 130.81 86.36) (diameter 0) (color 0 0 0 0)
   )
-  (junction (at 260.35 128.27) (diameter 0) (color 0 0 0 0)
-  )
   (junction (at 33.02 68.58) (diameter 0) (color 0 0 0 0)
   )
+  (no_connect (at 261.62 125.73))
   (no_connect (at 261.62 123.19))
   (no_connect (at 261.62 120.65))
@@
     (stroke (width 0) (type default))
   )
-  (wire (pts (xy 260.35 125.73) (xy 260.35 128.27))
-    (stroke (width 0) (type default))
-  )
   (wire (pts (xy 81.28 165.1) (xy 83.82 165.1))
     (stroke (width 0) (type default))
@@
     (stroke (width 0) (type default))
   )
-  (wire (pts (xy 259.08 128.27) (xy 260.35 128.27))
-    (stroke (width 0) (type default))
-  )
-  (wire (pts (xy 260.35 128.27) (xy 261.62 128.27))
+  (wire (pts (xy 259.08 128.27) (xy 261.62 128.27))
     (stroke (width 0) (type default))
   )
@@
     (stroke (width 0) (type default))
   )
-  (wire (pts (xy 261.62 125.73) (xy 260.35 125.73))
-    (stroke (width 0) (type default))
-  )
